File: GBDSO.sch (KiCad schematic (older format))
At the start: 66 parts, among them P1 100k, P2 100k, U1 TL062, U2 DS1267_SOIC, U3 TL062, U4 MAX114CAG, U5 74HC175D, U6 74HC138D, U7 AT27C256R, U8 TLC272, U9 MAX828

Commit message: updated schematic
Parts:
- added J1, J2: MJ-3523-SMT-TR, MJ-3523-SMT-TR:MJ-3523-SMT-TR, symbol MJ-3523-SMT-TR:MJ-3523-SMT-TR
- added SW1, SW2: SW_SPDT, Button_Switch_SMD:SW_SPDT_CK-JS102011SAQN, symbol Switch:SW_SPDT
Connections:
- net labels added: +5V, +5VA, +5VC, -5V, A0, A1, A10, A11, A12, A13, A14, A15, A2, A3, A4, A5, A6, A7, A8, A9, D0, D1, D2, D3, D4, D5, D6, D7, ECLK, GND, ~RD, ~WR
- wire segments 0 -> 112
Other:
- moved on the sheet: C1, C10, C11, C12, C13, C14, C15, C16, C17, C18, C19, C2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

Commit message: finished schematic, need to double check to be sure
Connections:
- net labels added: +2.5V, -2.5V
- wire segments 112 -> 368
- no-connect marks 0 -> 15
Other:
- moved on the sheet: C1, C10, C11, C12, C13, C14, C15, C16, C17, C18, C19, C2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

Commit message: updated schematic, corrected some errors
Connections:
- wire segments 368 -> 370
Other:
- moved on the sheet: U3A, U3B
Changed lines of the file:
@@
 L linear:TL062 U3
 U 1 1 5C60B392
+P 4520 4750
+F 0 "U3" H 4520 4950 50  0000 L CNN
+F 1 "TL062" H 4520 4550 50  0000 L CNN
+F 2 "Package_SO:SO-8_5.3x6.2mm_P1.27mm" H 4520 4750 50  0001 C CNN
+F 3 "" H 4520 4750 50  0001 C CNN
+	1    4520 4750
+	1    0    0    1
+$EndComp
+$Comp
+L linear:TL062 U3
+U 2 1 5C60B3F3
 P 2560 4170
 F 0 "U3" H 2560 4370 50  0000 L CNN
@@
 F 2 "Package_SO:SO-8_5.3x6.2mm_P1.27mm" H 2560 4170 50  0001 C CNN
 F 3 "" H 2560 4170 50  0001 C CNN
-	1    2560 4170
-	1    0    0    1
-$EndComp
-$Comp
-L linear:TL062 U3
-U 2 1 5C60B3F3
-P 4520 4750
-F 0 "U3" H 4520 4950 50  0000 L CNN
-F 1 "TL062" H 4520 4550 50  0000 L CNN
-F 2 "Package_SO:SO-8_5.3x6.2mm_P1.27mm" H 4520 4750 50  0001 C CNN
-F 3 "" H 4520 4750 50  0001 C CNN
-	2    4520 4750
+	2    2560 4170
 	1    0    0    1
 $EndComp
@@
 $EndComp
 $Comp
-L power:GND #PWR?
+L power:GND #PWR0101
 U 1 1 5C622ED2
 P 8450 2500
-F 0 "#PWR?" H 8450 2250 50  0001 C CNN
+F 0 "#PWR0101" H 8450 2250 50  0001 C CNN
 F 1 "GND" H 8455 2327 50  0000 C CNN
 F 2 "" H 8450 2500 50  0001 C CNN
@@
 	8450 2500 8450 2450
 $Comp
-L power:GND #PWR?
+L power:GND #PWR0102
 U 1 1 5C623302
 P 7700 5260
-F 0 "#PWR?" H 7700 5010 50  0001 C CNN
+F 0 "#PWR0102" H 7700 5010 50  0001 C CNN
 F 1 "GND" H 7705 5087 50  0000 C CNN
 F 2 "" H 7700 5260 50  0001 C CNN
@@
 	7700 5260 7700 5210
 $Comp
-L power:GND #PWR?
+L power:GND #PWR0103
 U 1 1 5C6238A8
 P 9350 6060
-F 0 "#PWR?" H 9350 5810 50  0001 C CNN
+F 0 "#PWR0103" H 9350 5810 50  0001 C CNN
 F 1 "GND" H 9355 5887 50  0000 C CNN
 F 2 "" H 9350 6060 50  0001 C CNN
@@
 ~RD
 $Comp
-L power:GND #PWR?
+L power:GND #PWR0104
 U 1 1 5C64CCD1
 P 630 7490
-F 0 "#PWR?" H 630 7240 50  0001 C CNN
+F 0 "#PWR0104" H 630 7240 50  0001 C CNN
 F 1 "GND" H 635 7317 50  0000 C CNN
 F 2 "" H 630 7490 50  0001 C CNN
@@
 Connection ~ 2480 6240
 $Comp
-L power:GND #PWR?
+L power:GND #PWR0105
 U 1 1 5C690775
 P 9700 3860
-F 0 "#PWR?" H 9700 3610 50  0001 C CNN
+F 0 "#PWR0105" H 9700 3610 50  0001 C CNN
 F 1 "GND" H 9705 3687 50  0000 C CNN
 F 2 "" H 9700 3860 50  0001 C CNN
@@
 	3650 7200 3650 7150
 $Comp
-L power:GND #PWR?
+L power:GND #PWR0106
 U 1 1 5C6DF12D
 P 3150 7250
-F 0 "#PWR?" H 3150 7000 50  0001 C CNN
+F 0 "#PWR0106" H 3150 7000 50  0001 C CNN
 F 1 "GND" H 3155 7077 50  0000 C CNN
 F 2 "" H 3150 7250 50  0001 C CNN
@@
 	7700 3810 7700 3910
 $Comp
-L power:GND #PWR?
+L power:GND #PWR0107
 U 1 1 5C742DD7
 P 8100 3910
-F 0 "#PWR?" H 8100 3660 50  0001 C CNN
+F 0 "#PWR0107" H 8100 3660 50  0001 C CNN
 F 1 "GND" H 8105 3737 50  0000 C CNN
 F 2 "" H 8100 3910 50  0001 C CNN
@@
 	8450 900  8450 950
 $Comp
-L power:GND #PWR?
+L power:GND #PWR0108
 U 1 1 5C75E1DA
 P 8850 950
-F 0 "#PWR?" H 8850 700 50  0001 C CNN
+F 0 "#PWR0108" H 8850 700 50  0001 C CNN
 F 1 "GND" H 8855 777 50  0000 C CNN
 F 2 "" H 8850 950 50  0001 C CNN
@@
 	8850 900  8750 900
 $Comp
-L power:GND #PWR?
+L power:GND #PWR0109
 U 1 1 5C772D46
 P 5770 3020
-F 0 "#PWR?" H 5770 2770 50  0001 C CNN
+F 0 "#PWR0109" H 5770 2770 50  0001 C CNN
 F 1 "GND" H 5775 2847 50  0000 C CNN
 F 2 "" H 5770 3020 50  0001 C CNN
@@
 $EndComp
 $Comp
-L power:GND #PWR?
+L power:GND #PWR0110
 U 1 1 5C63831F
 P 730 2530
-F 0 "#PWR?" H 730 2280 50  0001 C CNN
+F 0 "#PWR0110" H 730 2280 50  0001 C CNN
 F 1 "GND" H 735 2357 50  0000 C CNN
 F 2 "" H 730 2530 50  0001 C CNN
@@
 	1280 1350 1280 1630
 Wire Wire Line
-	2050 4430 2050 4450
-Wire Wire Line
 	2050 4450 1870 4450
 Wire Wire Line
 	1870 4450 1870 4470
-Connection ~ 2050 4450
-Wire Wire Line
-	2050 4450 2050 4470
 Wire Wire Line
 	2010 4070 2050 4070
@@
 Connection ~ 1350 4840
 $Comp
-L power:GND #PWR?
+L power:GND #PWR0111
 U 1 1 5C82F092
 P 870 4870
-F 0 "#PWR?" H 870 4620 50  0001 C CNN
+F 0 "#PWR0111" H 870 4620 50  0001 C CNN
 F 1 "GND" H 875 4697 50  0000 C CNN
 F 2 "" H 870 4870 50  0001 C CNN
@@
 	6060 6930 6090 6930
 $Comp
-L power:GND #PWR?
+L power:GND #PWR0112
 U 1 1 5C6E7C14
 P 6100 7170
-F 0 "#PWR?" H 6100 6920 50  0001 C CNN
+F 0 "#PWR0112" H 6100 6920 50  0001 C CNN
 F 1 "GND" H 6105 6997 50  0000 C CNN
 F 2 "" H 6100 7170 50  0001 C CNN
@@
 Connection ~ 6700 5980
 $Comp
-L power:GND #PWR?
+L power:GND #PWR0113
 U 1 1 5C77BD37
 P 6700 6290
-F 0 "#PWR?" H 6700 6040 50  0001 C CNN
+F 0 "#PWR0113" H 6700 6040 50  0001 C CNN
 F 1 "GND" H 6705 6117 50  0000 C CNN
 F 2 "" H 6700 6290 50  0001 C CNN
@@
 $EndComp
 $Comp
-L power:GND #PWR?
+L power:GND #PWR0114
 U 1 1 5C77C1AF
 P 5940 6290
-F 0 "#PWR?" H 5940 6040 50  0001 C CNN
+F 0 "#PWR0114" H 5940 6040 50  0001 C CNN
 F 1 "GND" H 5945 6117 50  0000 C CNN
 F 2 "" H 5940 6290 50  0001 C CNN
@@
 	5940 5980 5940 6050
 $Comp
-L power:GND #PWR?
+L power:GND #PWR0115
 U 1 1 5C7B9164
 P 4630 7470
-F 0 "#PWR?" H 4630 7220 50  0001 C CNN
+F 0 "#PWR0115" H 4630 7220 50  0001 C CNN
 F 1 "GND" H 4635 7297 50  0000 C CNN
 F 2 "" H 4630 7470 50  0001 C CNN
@@
 	6540 1070 6450 1070
 $Comp
-L power:GND #PWR?
+L power:GND #PWR0116
 U 1 1 5C9F7031
 P 6820 1120
-F 0 "#PWR?" H 6820 870 50  0001 C CNN
+F 0 "#PWR0116" H 6820 870 50  0001 C CNN
 F 1 "GND" H 6825 947 50  0000 C CNN
 F 2 "" H 6820 1120 50  0001 C CNN
@@
 NoConn ~ 7200 4210
 $Comp
-L power:GND #PWR?
+L power:GND #PWR0117
 U 1 1 5CD9E116
 P 4410 3590
-F 0 "#PWR?" H 4410 3340 50  0001 C CNN
+F 0 "#PWR0117" H 4410 3340 50  0001 C CNN
 F 1 "GND" H 4415 3417 50  0000 C CNN
 F 2 "" H 4410 3590 50  0001 C CNN
@@
 	4110 3880 4110 3800
 $Comp
-L power:GND #PWR?
+L power:GND #PWR0118
 U 1 1 5CDE026A
 P 4750 2310
-F 0 "#PWR?" H 4750 2060 50  0001 C CNN
+F 0 "#PWR0118" H 4750 2060 50  0001 C CNN
 F 1 "GND" H 4755 2137 50  0000 C CNN
 F 2 "" H 4750 2310 50  0001 C CNN
@@
 	10870 1670 10870 1560
 $Comp
-L power:GND #PWR?
+L power:GND #PWR0119
 U 1 1 5CEF24FE
 P 10640 1690
-F 0 "#PWR?" H 10640 1440 50  0001 C CNN
+F 0 "#PWR0119" H 10640 1440 50  0001 C CNN
 F 1 "GND" H 10645 1517 50  0000 C CNN
 F 2 "" H 10640 1690 50  0001 C CNN
@@
 Wire Wire Line
 	4460 850  4460 910
-Text GLabel 2430 2100 3    50   Input ~ 0
+Text GLabel 4530 1560 2    50   Input ~ 0
 -5V
-Text GLabel 2460 4520 3    50   Input ~ 0
+Text GLabel 4500 4380 2    50   Input ~ 0
 -5V
 Text GLabel 4420 5110 3    50   Input ~ 0
@@
 	4010 2900 3820 2900
 Wire Wire Line
-	2430 2100 2430 2030
-Wire Wire Line
 	4890 1210 4860 1210
 Wire Wire Line
@@
 Connection ~ 4160 1630
 $Comp
-L power:GND #PWR?
+L power:GND #PWR0120
 U 1 1 5D497178
 P 4010 1060
-F 0 "#PWR?" H 4010 810 50  0001 C CNN
+F 0 "#PWR0120" H 4010 810 50  0001 C CNN
 F 1 "GND" H 4015 887 50  0000 C CNN
 F 2 "" H 4010 1060 50  0001 C CNN
@@
 	5250 840  5250 880
 $Comp
-L power:GND #PWR?
+L power:GND #PWR0121
 U 1 1 5D5721B6
 P 5250 1480
-F 0 "#PWR?" H 5250 1230 50  0001 C CNN
+F 0 "#PWR0121" H 5250 1230 50  0001 C CNN
 F 1 "GND" H 5255 1307 50  0000 C CNN
 F 2 "" H 5250 1480 50  0001 C CNN
@@
 	5500 1810 5850 1810
 Wire Wire Line
-	2460 4520 2460 4470
-Wire Wire Line
 	4820 4750 4850 4750
 Wire Wire Line
@@
 Connection ~ 5210 4750
 $Comp
-L power:GND #PWR?
+L power:GND #PWR0122
 U 1 1 5D6B7A30
 P 5210 5040
-F 0 "#PWR?" H 5210 4790 50  0001 C CNN
+F 0 "#PWR0122" H 5210 4790 50  0001 C CNN
 F 1 "GND" H 5215 4867 50  0000 C CNN
 F 2 "" H 5210 5040 50  0001 C CNN
@@
 	5550 4750 5210 4750
 $Comp
-L power:GND #PWR?
+L power:GND #PWR0123
 U 1 1 5D7621C5
 P 4050 4990
-F 0 "#PWR?" H 4050 4740 50  0001 C CNN
+F 0 "#PWR0123" H 4050 4740 50  0001 C CNN
 F 1 "GND" H 4055 4817 50  0000 C CNN
 F 2 "" H 4050 4990 50  0001 C CNN
@@
 	3690 4650 3820 4650
 Connection ~ 3820 4650
+Wire Wire Line
+	4530 1560 4460 1560
+Wire Wire Line
+	4460 1560 4460 1510
+Wire Wire Line
+	4500 4380 4420 4380
+Wire Wire Line
+	4420 4380 4420 4450
+Wire Wire Line
+	2050 4450 2050 4470
+Wire Wire Line
+	2050 4450 2050 4420
 Wire Bus Line
 	5370 2670 5370 3310
@@
 Wire Bus Line
 	10150 4310 10150 6460
+Connection ~ 2050 4450
 $EndSCHEMATC

Commit message: updated schematic, new generated netlist, finished pcb
Parts:
- added J3: Conn_01x32, GB_EdgeConnector:GB_EdgeConnector, symbol Connector_Generic:Conn_01x32
Connections:
- wire segments 370 -> 401
- no-connect marks 15 -> 18
Changed lines of the file:
@@
 Wire Wire Line
 	2050 4450 2050 4420
+Connection ~ 2050 4450
+$Comp
+L Connector_Generic:Conn_01x32 J3
+U 1 1 5C696C85
+P 10790 4770
+F 0 "J3" H 10870 4762 50  0000 L CNN
+F 1 "Conn_01x32" H 10870 4671 50  0000 L CNN
+F 2 "GB_EdgeConnector:GB_EdgeConnector" H 10790 4770 50  0001 C CNN
+F 3 "~" H 10790 4770 50  0001 C CNN
+	1    10790 4770
+	1    0    0    -1
+$EndComp
+Text GLabel 10550 3220 1    50   Input ~ 0
++5V
+Wire Wire Line
+	10550 3220 10550 3270
+Wire Wire Line
+	10550 3270 10590 3270
+Entry Wire Line
+	10150 3470 10250 3370
+Wire Wire Line
+	10250 3370 10590 3370
+Entry Wire Line
+	10150 3570 10250 3470
+Wire Wire Line
+	10250 3470 10590 3470
+Entry Wire Line
+	10150 3670 10250 3570
+Wire Wire Line
+	10250 3570 10590 3570
+Entry Wire Line
+	10150 3870 10250 3770
+Entry Wire Line
+	10150 3970 10250 3870
+Entry Wire Line
+	10150 4070 10250 3970
+Entry Wire Line
+	10150 4170 10250 4070
+Entry Wire Line
+	10150 4270 10250 4170
+Entry Wire Line
+	10150 4370 10250 4270
+Entry Wire Line
+	10150 4470 10250 4370
+Entry Wire Line
+	10150 4570 10250 4470
+Entry Wire Line
+	10150 4670 10250 4570
+Entry Wire Line
+	10150 4770 10250 4670
+Entry Wire Line
+	10150 4870 10250 4770
+Entry Wire Line
+	10150 4970 10250 4870
+Entry Wire Line
+	10150 5070 10250 4970
+Entry Wire Line
+	10150 5170 10250 5070
+Entry Wire Line
+	10150 5270 10250 5170
+Entry Wire Line
+	10150 5370 10250 5270
+Wire Wire Line
+	10250 5270 10590 5270
+Entry Wire Line
+	10150 5470 10250 5370
+Entry Wire Line
+	10150 5570 10250 5470
+Entry Wire Line
+	10150 5670 10250 5570
+Entry Wire Line
+	10150 5770 10250 5670
+Entry Wire Line
+	10150 5870 10250 5770
+Entry Wire Line
+	10150 5970 10250 5870
+Entry Wire Line
+	10150 6070 10250 5970
+Entry Wire Line
+	10150 6170 10250 6070
+$Comp
+L power:GND #PWR0124
+U 1 1 5CBE744A
+P 10530 6410
+F 0 "#PWR0124" H 10530 6160 50  0001 C CNN
+F 1 "GND" H 10535 6237 50  0000 C CNN
+F 2 "" H 10530 6410 50  0001 C CNN
+F 3 "" H 10530 6410 50  0001 C CNN
+	1    10530 6410
+	1    0    0    -1
+$EndComp
+Wire Wire Line
+	10530 6410 10530 6370
+Wire Wire Line
+	10530 6370 10590 6370
+Text Label 10390 5370 0    50   ~ 0
+D0
+Text Label 10390 5470 0    50   ~ 0
+D1
+Text Label 10390 5570 0    50   ~ 0
+D2
+Text Label 10390 5670 0    50   ~ 0
+D3
+Text Label 10390 5770 0    50   ~ 0
+D4
+Text Label 10390 5870 0    50   ~ 0
+D5
+Text Label 10390 5970 0    50   ~ 0
+D6
+Text Label 10390 6070 0    50   ~ 0
+D7
+Wire Wire Line
+	10250 5370 10590 5370
+Wire Wire Line
+	10250 5470 10590 5470
+Wire Wire Line
+	10250 5570 10590 5570
+Wire Wire Line
+	10250 5670 10590 5670
+Wire Wire Line
+	10250 5770 10590 5770
+Wire Wire Line
+	10250 5870 10590 5870
+Wire Wire Line
+	10250 5970 10590 5970
+Wire Wire Line
+	10250 6070 10590 6070
+Text Label 10390 3770 0    50   ~ 0
+A0
+Text Label 10390 3870 0    50   ~ 0
+A1
+Text Label 10390 3970 0    50   ~ 0
+A2
+Text Label 10390 4070 0    50   ~ 0
+A3
+Text Label 10390 4170 0    50   ~ 0
+A4
+Text Label 10390 4270 0    50   ~ 0
+A5
+Text Label 10390 4370 0    50   ~ 0
+A6
+Text Label 10390 4470 0    50   ~ 0
+A7
+Text Label 10390 4570 0    50   ~ 0
+A8
+Text Label 10390 4670 0    50   ~ 0
+A9
+Text Label 10390 4770 0    50   ~ 0
+A10
+Text Label 10390 4870 0    50   ~ 0
+A11
+Text Label 10390 4970 0    50   ~ 0
+A12
+Text Label 10390 5070 0    50   ~ 0
+A13
+Text Label 10390 5170 0    50   ~ 0
+A14
+Wire Wire Line
+	10250 5170 10590 5170
+Wire Wire Line
+	10250 5070 10590 5070
+Wire Wire Line
+	10250 4970 10590 4970
+Wire Wire Line
+	10250 4870 10590 4870
+Wire Wire Line
+	10250 4770 10590 4770
+Wire Wire Line
+	10250 4270 10590 4270
+Wire Wire Line
+	10250 4370 10590 4370
+Wire Wire Line
+	10250 4470 10590 4470
+Wire Wire Line
+	10250 4570 10590 4570
+Wire Wire Line
+	10250 4670 10590 4670
+Wire Wire Line
+	10250 4070 10590 4070
+Wire Wire Line
+	10250 4170 10590 4170
+Wire Wire Line
+	10250 3770 10590 3770
+Wire Wire Line
+	10250 3870 10590 3870
+Wire Wire Line
+	10250 3970 10590 3970
+Text Label 10360 3370 0    50   ~ 0
+ECLK
+Text Label 10370 3570 0    50   ~ 0
+~RD
+Text Label 10370 3470 0    50   ~ 0
+~WR
+Text Label 10390 5270 0    50   ~ 0
+A15
+NoConn ~ 10590 6270
+NoConn ~ 10590 6170
+NoConn ~ 10590 3670
 Wire Bus Line
 	5370 2670 5370 3310
@@
 	8450 3310 8450 6460
 Wire Bus Line
-	10150 4310 10150 6460
-Connection ~ 2050 4450
+	10150 3340 10150 6460
 $EndSCHEMATC

Commit message: general update and lib fix + new generated gerber
Parts:
- added unit 3 of U1
- added unit 3 of U3
- D1, D2: symbol bav199:BAV199 -> BAV199:BAV199
- U1, U3: symbol linear:TL062 -> Amplifier_Operational:TL062
- U2: symbol maxim:DS1267_SOIC -> Potentiometer_Digital:DS1267_SOIC
Other:
- note added: "04/03/2019"
- note added: "Game Boy Oscilloscope in KiCAD"
Changed lines of the file:
@@
 $EndDescr
 $Comp
-L linear:TL062 U1
+L Amplifier_Operational:TL062 U1
 U 1 1 5C60B30E
 P 4560 1210
@@
 $EndComp
 $Comp
-L linear:TL062 U1
+L Amplifier_Operational:TL062 U1
 U 2 1 5C60B373
 P 2530 1730
@@
 $EndComp
 $Comp
-L linear:TL062 U3
+L Amplifier_Operational:TL062 U3
 U 1 1 5C60B392
 P 4520 4750
@@
 $EndComp
 $Comp
-L linear:TL062 U3
+L Amplifier_Operational:TL062 U3
 U 2 1 5C60B3F3
 P 2560 4170
@@
 $EndComp
 $Comp
-L maxim:DS1267_SOIC U2
+L Potentiometer_Digital:DS1267_SOIC U2
 U 1 1 5C60B43A
 P 4410 3000
@@
 $EndComp
 $Comp
-L bav199:BAV199 D1
+L BAV199:BAV199 D1
 U 1 1 5C61AAEF
 P 1980 930
@@
 $EndComp
 $Comp
-L bav199:BAV199 D2
+L BAV199:BAV199 D2
 U 1 1 5C62C724
 P 2090 3320
@@
 NoConn ~ 4810 3100
 NoConn ~ 4810 3200
-Text GLabel 4460 850  1    50   Input ~ 0
+Text GLabel 3290 1310 1    50   Input ~ 0
 +5VA
 Wire Wire Line
-	4460 850  4460 910
-Text GLabel 4530 1560 2    50   Input ~ 0
+	3290 1310 3290 1370
+Text GLabel 3360 2020 2    50   Input ~ 0
 -5V
-Text GLabel 4500 4380 2    50   Input ~ 0
+Text GLabel 3170 4620 0    50   Input ~ 0
 -5V
-Text GLabel 4420 5110 3    50   Input ~ 0
+Text GLabel 3250 3890 1    50   Input ~ 0
 +5VA
 Wire Wire Line
-	4420 5110 4420 5050
+	3250 3890 3250 3950
 Wire Wire Line
 	4010 2800 3700 2800
@@
 Connection ~ 3820 4650
 Wire Wire Line
-	4530 1560 4460 1560
-Wire Wire Line
-	4460 1560 4460 1510
-Wire Wire Line
-	4500 4380 4420 4380
-Wire Wire Line
-	4420 4380 4420 4450
+	3360 2020 3290 2020
+Wire Wire Line
+	3290 2020 3290 1970
+Wire Wire Line
+	3170 4620 3250 4620
+Wire Wire Line
+	3250 4620 3250 4550
 Wire Wire Line
 	2050 4450 2050 4470
@@
 NoConn ~ 10590 6170
 NoConn ~ 10590 3670
+$Comp
+L Amplifier_Operational:TL062 U1
+U 3 1 5C833BB5
+P 3390 1670
+F 0 "U1" H 3348 1716 50  0000 L CNN
+F 1 "TL062" H 3348 1625 50  0000 L CNN
+F 2 "" H 3390 1670 50  0001 C CNN
+F 3 "http://www.ti.com/lit/ds/symlink/tl061.pdf" H 3390 1670 50  0001 C CNN
+	3    3390 1670
+	1    0    0    -1
+$EndComp
+$Comp
+L Amplifier_Operational:TL062 U3
+U 3 1 5C833D27
+P 3350 4250
+F 0 "U3" H 3308 4296 50  0000 L CNN
+F 1 "TL062" H 3308 4205 50  0000 L CNN
+F 2 "" H 3350 4250 50  0001 C CNN
+F 3 "http://www.ti.com/lit/ds/symlink/tl061.pdf" H 3350 4250 50  0001 C CNN
+	3    3350 4250
+	1    0    0    -1
+$EndComp
+Text Notes 7380 7500 0    50   ~ 0
+Game Boy Oscilloscope in KiCAD
+Text Notes 8140 7640 0    50   ~ 0
+04/03/2019
 Wire Bus Line
 	5370 2670 5370 3310
