File: GBDSO EPROM Adapter Board.sch (KiCad schematic (older format))
At the start: 2 parts, among them J4 GameBoy Cartridge Connector, U10 AT27C256R-PDIP28

Commit message: updated schematic, pcb, pictures and readme because I changed the GB connector to the Xunbeifang one
Parts:
- J4: footprint Gekkio_Connector_PCBEdge:GameBoy_Cartridge_DSLite_1x32_P1.50mm_Socket_Horizontal -> Game_Boy_Cartridge_Slot_Xunbeifang_GNI172:Game_Boy_Cartridge_Slot_Xunbeifang_GNI172
Changed lines of the file:
@@
 F 0 "J4" H 6710 5210 50  0000 L CNN
 F 1 "GameBoy Cartridge Connector" V 6880 3330 50  0000 L CNN
-F 2 "Gekkio_Connector_PCBEdge:GameBoy_Cartridge_DSLite_1x32_P1.50mm_Socket_Horizontal" H 6740 3600 50  0001 C CNN
+F 2 "Game_Boy_Cartridge_Slot_Xunbeifang_GNI172:Game_Boy_Cartridge_Slot_Xunbeifang_GNI172" H 6740 3600 50  0001 C CNN
 F 3 "~" H 6740 3600 50  0001 C CNN
 	1    6740 3600
